Commit message: added comments

File: install/argo_sim/share/argo_sim/description/urdf/argo.urdf.xacro (robot description, xacro)
@@ -172,4 +172,5 @@
             <remapping>~/out:=${prefix}_laser/scan</remapping>
           </ros>
+          <frame_name>${prefix}_laser_link</frame_name>
           <frameName>${prefix}_laser_link</frameName>
           <output_type>sensor_msgs/LaserScan</output_type>
@@ -271,5 +272,5 @@
     <joint name="IMU_joint" type="fixed">
       <axis xyz="0 0 1" />
-      <origin xyz="0 0 ${top_platform}" rpy="0 0 ${pi/2}"/>
+      <origin xyz="0 0 ${top_platform}" rpy="0 0 0"/>
       <parent link="base_link"/>
       <child link="imu_link"/>
